File: cortex_main.kicad_pcb (KiCad board)
At the start: 2 copper layers, 141 x 129.5 mm, 52 parts, among them J1 TEST_1P, J2 TEST_1P, P1 CONN_01X04, P10 CONN_01X03, P11 CONN_01X03, P12 CONN_01X03, P13 CONN_01X03, P14 CONN_01X03, P15 CONN_01X03, P16 CONN_01X02, P17 CONN_01X02, P18 CONN_01X02, P19 CONN_01X02, P2 CONN_02X04, P20 CONN_01X03, P21 CONN_01X02, P22 CONN_01X02, P23 CONN_01X02, P24 CONN_01X02, P25 CONN_01X02, P3 CONN_01X02, P4 CONN_01X04, P5 CONN_01X02, P6 CONN_01X06, P7 CONN_01X06, P8 CONN_01X03, P9 CONN_01X03, Q1 IRF540N, Q2 IRF540N, Q3 IRF540N, Q4 IRF540N, Q5 IRF540N, Q6 IRF540N, U1 socket_leon_x3_dil64, U2 socket_pololu_24v12, U3 socket_pololu_24v12, U4 socket_lm2596_mod, U5 socket_ams1117-3V3_mod, U6 MCP100-D

Commit message: cortex: add gnd test pad and text on PCB
Signed-off-by: Yannick Gicquel <ygicquel@gmail.com>
Parts:
- added J3: TEST_1P, Pin_Headers:Pin_Header_Straight_1x01_Pitch2.54mm, F.Cu at (43.2, 130.8)
Routing:
- added copper zone on B.Cu, net OUTP_ARMMOTOR_L
Other:
- board text added: "Cortex Bot 2017 V1"
Changed lines of the file:
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@@
 (kicad_pcb (version 4) (host pcbnew 4.0.6-e0-6349~53~ubuntu16.04.1)
   (general
-    (links 150)
-    (no_connects 21)
-    (area 32.944999 26.715 174.065001 157.555001)
+    (links 151)
+    (no_connects 20)
+    (area 32.944999 27.864999 174.065001 157.555001)
     (thickness 1.6)
-    (drawings 8)
+    (drawings 9)
     (tracks 252)
     (zones 0)
-    (modules 52)
+    (modules 53)
     (nets 84)
   )
@@
     )
   )
+  (module Pin_Headers:Pin_Header_Straight_1x01_Pitch2.54mm (layer F.Cu)
+    (at 43.18 130.81)
+    (descr "Through hole straight pin header, 1x01, 2.54mm pitch, single row")
+    (tags "Through hole pin header THT 1x01 2.54mm single row")
+    (fp_text reference J3 (at 0 -2.39) (layer F.SilkS)
+      (effects (font (size 1 1) (thickness 0.15)))
+    )
+    (fp_text value TEST_1P (at 0 2.39) (layer F.Fab)
+      (effects (font (size 1 1) (thickness 0.15)))
+    )
+    (fp_line (start -1.27 -1.27) (end -1.27 1.27) (layer F.Fab) (width 0.1))
+    (fp_line (start -1.27 1.27) (end 1.27 1.27) (layer F.Fab) (width 0.1))
+    (fp_line (start 1.27 1.27) (end 1.27 -1.27) (layer F.Fab) (width 0.1))
+    (fp_line (start 1.27 -1.27) (end -1.27 -1.27) (layer F.Fab) (width 0.1))
+    (fp_line (start -1.39 1.27) (end -1.39 1.39) (layer F.SilkS) (width 0.12))
+    (fp_line (start -1.39 1.39) (end 1.39 1.39) (layer F.SilkS) (width 0.12))
+    (fp_line (start 1.39 1.39) (end 1.39 1.27) (layer F.SilkS) (width 0.12))
+    (fp_line (start 1.39 1.27) (end -1.39 1.27) (layer F.SilkS) (width 0.12))
+    (fp_line (start -1.39 0) (end -1.39 -1.39) (layer F.SilkS) (width 0.12))
+    (fp_line (start -1.39 -1.39) (end 0 -1.39) (layer F.SilkS) (width 0.12))
+    (fp_line (start -1.6 -1.6) (end -1.6 1.6) (layer F.CrtYd) (width 0.05))
+    (fp_line (start -1.6 1.6) (end 1.6 1.6) (layer F.CrtYd) (width 0.05))
+    (fp_line (start 1.6 1.6) (end 1.6 -1.6) (layer F.CrtYd) (width 0.05))
+    (fp_line (start 1.6 -1.6) (end -1.6 -1.6) (layer F.CrtYd) (width 0.05))
+    (pad 1 thru_hole rect (at 0 0) (size 1.7 1.7) (drill 1) (layers *.Cu *.Mask)
+      (net 24 GND))
+    (model Pin_Headers.3dshapes/Pin_Header_Straight_1x01_Pitch2.54mm.wrl
+      (at (xyz 0 0 0))
+      (scale (xyz 1 1 1))
+      (rotate (xyz 0 0 90))
+    )
+  )
+  (gr_text "Cortex Bot\n2017\nV1" (at 162.56 149.86 270) (layer B.Cu)
+    (effects (font (size 3.5 3.5) (thickness 0.5)) (justify left mirror))
+  )
   (gr_line (start 173.99 27.94) (end 173.99 157.48) (angle 90) (layer Edge.Cuts) (width 0.15))
   (gr_line (start 33.02 157.48) (end 173.99 157.48) (angle 90) (layer Edge.Cuts) (width 0.15))
@@
   (segment (start 110.49 31.75) (end 86.36 31.75) (width 3) (layer B.Cu) (net 23))
   (segment (start 114.3 35.56) (end 110.49 31.75) (width 3) (layer B.Cu) (net 23))
-  (segment (start 102.87 106.68) (end 102.87 101.6) (width 0.75) (layer F.Cu) (net 24) (status C00000))
-  (segment (start 83.82 114.3) (end 82.55 114.3) (width 0.75) (layer B.Cu) (net 24) (status 400000))
-  (segment (start 73.66 116.84) (end 73.66 120.65) (width 0.75) (layer B.Cu) (net 24) (status 800000))
+  (segment (start 102.87 106.68) (end 102.87 101.6) (width 0.75) (layer F.Cu) (net 24))
+  (segment (start 83.82 114.3) (end 82.55 114.3) (width 0.75) (layer B.Cu) (net 24))
+  (segment (start 73.66 116.84) (end 73.66 120.65) (width 0.75) (layer B.Cu) (net 24))
   (via (at 73.66 116.84) (size 1.6) (drill 0.8) (layers F.Cu B.Cu) (net 24))
   (segment (start 81.28 116.84) (end 73.66 116.84) (width 0.75) (layer F.Cu) (net 24))
@@
   (segment (start 69.85 109.22) (end 68.58 110.49) (width 0.75) (layer B.Cu) (net 44))
   (segment (start 68.58 110.49) (end 68.58 120.65) (width 0.75) (layer B.Cu) (net 44))
-  (segment (start 76.2 120.65) (end 76.2 115.57) (width 0.75) (layer B.Cu) (net 46) (status 400000))
-  (segment (start 74.93 114.3) (end 71.12 114.3) (width 0.75) (layer B.Cu) (net 46) (status 800000))
+  (segment (start 76.2 120.65) (end 76.2 115.57) (width 0.75) (layer B.Cu) (net 46))
+  (segment (start 74.93 114.3) (end 71.12 114.3) (width 0.75) (layer B.Cu) (net 46))
   (segment (start 76.2 115.57) (end 74.93 114.3) (width 0.75) (layer B.Cu) (net 46))
   (segment (start 127 143.51) (end 127 140.97) (width 0.75) (layer B.Cu) (net 47))
@@
     (polygon
       (pts
-        (xy 42.545 55.245) (xy 61.595 55.245) (xy 61.595 49.53) (xy 67.945 49.53) (xy 67.945 55.245)
-        (xy 88.9 55.245) (xy 88.9 35.56) (xy 102.87 35.56) (xy 102.87 48.26) (xy 102.87 59.69)
-        (xy 102.87 64.77) (xy 85.09 64.77) (xy 85.09 77.47) (xy 65.405 77.47) (xy 65.405 82.55)
-        (xy 61.595 82.55) (xy 61.595 77.47) (xy 40.005 77.47) (xy 40.005 82.55) (xy 35.56 82.55)
-        (xy 35.56 49.53) (xy 42.545 49.53)
+        (xy 156.21 39.37) (xy 152.4 39.37) (xy 152.4 154.94) (xy 35.56 154.94) (xy 35.56 83.82)
+        (xy 88.9 83.82) (xy 88.9 67.31) (xy 88.9 64.77) (xy 85.09 64.77) (xy 85.09 77.47)
+        (xy 65.405 77.47) (xy 65.405 82.55) (xy 61.595 82.55) (xy 61.595 77.47) (xy 40.005 77.47)
+        (xy 40.005 82.55) (xy 35.56 82.55) (xy 35.56 49.53) (xy 42.545 49.53) (xy 42.545 55.245)
+        (xy 61.595 55.245) (xy 61.595 49.53) (xy 67.945 49.53) (xy 67.945 55.245) (xy 88.9 55.245)
+        (xy 88.9 35.56) (xy 102.87 35.56) (xy 102.87 30.48) (xy 156.21 30.48)
       )
     )
@@
     )
   )
-  (zone (net 24) (net_name GND) (layer B.Cu) (hatch edge 0.508)
+  (zone (net 65) (net_name OUTP_ARMMOTOR_L) (layer B.Cu) (hatch edge 0.508)
     (connect_pads yes (clearance 1.016))
     (min_thickness 0.254)
@@
     (polygon
       (pts
-        (xy 156.21 39.37) (xy 152.4 39.37) (xy 152.4 154.94) (xy 35.56 154.94) (xy 35.56 83.82)
-        (xy 88.9 83.82) (xy 88.9 67.31) (xy 106.68 67.31) (xy 106.68 46.99) (xy 106.68 30.48)
-        (xy 156.21 30.48)
+        (xy 171.45 39.37) (xy 171.45 110.49) (xy 161.29 110.49) (xy 161.29 106.68) (xy 166.37 106.68)
+        (xy 166.37 97.79) (xy 161.29 97.79) (xy 161.29 93.98) (xy 166.37 93.98) (xy 166.37 82.55)
+        (xy 161.29 82.55) (xy 161.29 78.74) (xy 166.37 78.74) (xy 166.37 69.85) (xy 161.29 69.85)
+        (xy 161.29 66.04) (xy 166.37 66.04) (xy 166.37 57.15) (xy 161.29 57.15) (xy 161.29 53.34)
+        (xy 166.37 53.34) (xy 166.37 44.45) (xy 161.29 44.45) (xy 161.29 40.64) (xy 158.75 35.56)
+        (xy 158.75 33.02) (xy 165.1 33.02)
       )
     )
